File: Teco.kicad_pcb (KiCad board)
At the start: 2 copper layers, 54 parts, among them Q1 BC848, Q2 BC807, Q3 IRLML9303, SW1 SWITCH_2x

Commit message: Sch updated Layout done
Parts:
- removed C2: 0.1u, Capacitors:CAP_0603
- removed F1: Fuse0R, Resistors:RES_0603_FUSE
- removed HOLE1, HOLE2, HOLE3, HOLE4: HOLE_METALLED, PCB:Hole2d4_out4d5mm
- removed R3: 100k, Resistors:RES_0603
- removed R8: DNM, Resistors:RES_0603
- added C12: 0.1u, Capacitors:CAP_0603, B.Cu at (142.0, 89.0)
- added C13: 10n, Capacitors:CAP_0603, B.Cu at (117.8, 91.7)
- added D4: PMEG2020, Diodes:SOD323, B.Cu at (141.8, 93.2)
- added L1: BLM15AG102, Inductors:IND_0402, B.Cu at (120.0, 90.2)
- added L2: BLM15AG102, Inductors:IND_0402, B.Cu at (120.0, 93.4)
- added R23: 1M, Resistors:RES_0603, B.Cu at (141.3, 91.7)
- C1, C10, C11, C3, C4, C5, C6, C7, C8, C9, DA1, DD1, Q1, Q3, R1, R10, R17, R18, R19, R2, R20, R21, R22, R4, R5, R6, R7, R9, XL1, XTAL1: moved to B.Cu
- Q2: value BC807 -> BC848; moved to B.Cu
- R12: value 1k -> 10k; moved to B.Cu
- R13: value 5R1 -> 10k; moved to B.Cu
- R14: value 1k -> 100k; moved to B.Cu
- SW1: value SWITCH_2x -> BUTTON; footprint BtnsSwitches:BTN_PSM6 -> BtnsSwitches:BTN_4x4_SMD
- moved C6 137.4 mm to (122.8, 79.0), turned to 270 degrees
- moved D2 135.4 mm to (127.3, 77.8), turned to 180 degrees
- moved R16 135.3 mm to (127.2, 75.4), turned to 180 degrees
- moved R2 134.5 mm to (120.6, 75.4), turned to 180 degrees
- moved D3 133.5 mm to (131.2, 73.4), turned to 180 degrees
- moved R1 128.5 mm to (122.8, 84.3), turned to 90 degrees
- moved C9 127.3 mm to (122.6, 91.3), turned to 180 degrees
- moved C8 126.0 mm to (122.6, 89.0), turned to 180 degrees
- moved R15 125.9 mm to (127.3, 81.0), turned to 180 degrees
- moved R9 124.9 mm to (137.2, 78.1), turned to 90 degrees
- moved R4 124.9 mm to (125.7, 75.4), turned to 180 degrees
- moved R10 124.6 mm to (137.2, 83.4), turned to 90 degrees
- moved C1 122.9 mm to (131.7, 74.8), turned to 90 degrees
- moved R5 121.4 mm to (136.6, 73.6), turned to 270 degrees
- moved C7 120.8 mm to (133.3, 74.8), turned to 90 degrees
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Connections:
- DD1 pad 3: Net-(DD1-Pad3) -> (no net)
- DD1 pad 7: Net-(C2-Pad1) -> (no net)
- Q2 pad 2: +3.3V -> GND
- Q3 pad 1: Net-(Q2-Pad3) -> Net-(Q3-Pad1)
- Q3 pad 2: Net-(Q3-Pad2) -> +3.3V
- Q3 pad 3: Net-(F1-Pad1) -> Net-(D4-PadA)
- R12 pad 1: GND -> +3.3V
- R13 pad 1: Net-(Q3-Pad2) -> Net-(Q3-Pad1)
- R13 pad 2: +3.3V -> Net-(Q2-Pad3)
- R14 pad 1: Net-(Q3-Pad2) -> Net-(D4-PadA)
- SW1 pad 1: (no net) -> Net-(Q3-Pad1)
- SW1 pad 2: Net-(F1-Pad1) -> Net-(C12-Pad1)
- XL1 pad 1: +5V -> /5VIN
- XL1 pad 4: GND -> /GNDIN
- XL1 pad 5: GND -> /GNDIN
Other:
- board outline added: 42 x 24 mm
- rule pad_to_mask_clearance: 0.2 -> 0.1
- board text added: "B"
- board text added: "G"

Commit message: Sent to production
Parts:
- XL3: footprint Connectors:PBS-6R -> Connectors:PBS-6R-MIRR; moved to B.Cu
- XL4: footprint Connectors:PBS-2R -> Connectors:PBS-2R-MIRR; moved to B.Cu
- moved Logo1 37.3 mm to (124.0, 88.5)
- moved R18 5.92 mm to (142.8, 86.4), turned to 90 degrees
- moved R17 5.48 mm to (142.8, 89.4), turned to 90 degrees
- moved R19 5.18 mm to (142.8, 83.4), turned to 90 degrees
- moved R22 5.14 mm to (142.8, 92.4), turned to 270 degrees
- moved R21 3.75 mm to (139.1, 75.9)
- moved D4 1.90 mm to (139.9, 93.2)
- moved R23 1.90 mm to (139.4, 91.7)
- moved Q3 1.10 mm to (135.8, 92.4)
- moved R15 0.90 mm to (128.1, 81.3), turned to 270 degrees
- moved C12 0.85 mm to (141.2, 89.3)
- moved C6 0.70 mm to (122.8, 78.3)
- moved R14 0.41 mm to (138.9, 90.0)
- moved R5 0.30 mm to (136.9, 73.6)
- moved R6 0.30 mm to (138.5, 73.6)
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Routing:
- net GND: track 0.00 -> 245.1 mm, vias 0 -> 47
- net +3.3V: track 0.00 -> 80.1 mm, vias 0 -> 7
- net +5V: track 0.00 -> 24.7 mm, vias 0 -> 2
- net Net-(Q3-Pad1): track 0.00 -> 22.4 mm, vias 0 -> 1
- net /EXTPWR: track 0.00 -> 22.4 mm, vias 0 -> 1
- net /T_JTCK: track 0.00 -> 22.1 mm, vias 0 -> 2
- net /T_JTMS: track 0.00 -> 21.5 mm, vias 0 -> 2
- net /T_NRST: track 0.00 -> 20.2 mm, vias 0 -> 2
- net Net-(C12-Pad1): track 0.00 -> 20.1 mm, vias 0 -> 1
- net /GNDIN: track 0.00 -> 16.7 mm, vias 0 -> 2
- net /TXD: track 0.00 -> 15.5 mm, vias 0 -> 1
- net /AIN1: track 0.00 -> 15.2 mm, vias 0 -> 2
- net /T_SWO: track 0.00 -> 14.9 mm, vias 0 -> 2
- net /USB_D+: track 0.00 -> 14.5 mm, vias 0 -> 2
- net /RXD: track 0.00 -> 14.3 mm, vias 0 -> 1
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- added copper zone on B.Cu, net GND
- added copper zone on F.Cu, net GND
Other:
- net class Default: clearance 0.2 -> 0.15; trace_width 0.25 -> 0.15; via_dia 0.8 -> 0.7; via_drill 0.4 -> 0.3
- net class Wide added: clearance 0.2, trace_width 0.5, via_dia 0.7, via_drill 0.3
- rule trace_clearance: 0.2 -> 0.15
- rule trace_min: 0.2 -> 0.15
- board text added: "+ SWCLK GND SWDIO RX TX"
- board text added: "Ostranna Teco v1"
- board text added: "SWO NRST"

Commit message: + V2
Parts:
- added R3: 100k, Resistors:RES_0603, F.Cu at (134.9, 86.9)
- added R8: 10k, Resistors:RES_0603, B.Cu at (138.9, 88.4)
- R17, R22: value 4k7 -> 10k
- R6: value 36k -> 30k
- moved R21 2.46 mm to (140.0, 73.6), turned to 270 degrees
- moved Q2 0.82 mm to (137.2, 85.9)
- moved C10 0.76 mm to (140.4, 85.0)
- moved XTAL1 0.70 mm to (140.0, 81.2)
- moved C11 0.61 mm to (139.5, 77.3)
- moved C4 0.60 mm to (135.6, 82.8)
- moved R10 0.60 mm to (137.2, 82.8)
- moved C7 0.17 mm to (133.1, 74.8)
- moved C1 0.17 mm to (131.5, 74.8)
- moved R5 0.09 mm to (136.8, 73.6)
- moved R6 0.09 mm to (138.4, 73.6)
- moved R7 0.09 mm to (135.2, 73.6)
Routing:
- net GND: track 245.1 -> 235.1 mm, vias 47 -> 46
- net /T_SWO: track 14.9 -> 17.1 mm
- net Net-(Q2-Pad3): track 5.12 -> 7.06 mm, vias 0 -> 2
- net Net-(D4-PadA): track 5.64 -> 7.24 mm
- net Net-(R21-Pad1): track 2.69 -> 3.65 mm
- net /TXD: track 15.5 -> 14.5 mm
- net +3.3V: track 80.1 -> 79.3 mm, vias 7 -> 8
- net Net-(Q2-Pad1): track 4.81 -> 5.62 mm
- net /LED_STLINK: track 10.9 -> 10.2 mm
Other:
- board text added: "Ostranna Teco v2"
- board text removed: "Ostranna Teco v1"
