File: Teco.kicad_pcb (KiCad board)
At the start: 2 copper layers, 42 x 24 mm, 56 parts, among them Q2 BC848, Q3 IRLML9303, SW1 BUTTON

Commit message: + Teco v4 + USB renum returned!
Parts:
- removed L2, L3: BLM18EG221SN1D, Inductors:IND_0603
- added C13: 10n, Capacitors:CAP_0603, B.Cu at (119.8, 89.7)
- added Q1: BC848, SOT:SOT23-3, B.Cu at (127.5, 74.7)
- R1: value 100R -> 10k
- moved R2 13.7 mm to (117.9, 89.7), turned to -90 degrees
- moved C2 13.6 mm to (116.0, 89.7), turned to 90 degrees
- moved R1 12.0 mm to (130.1, 74.8), turned to -90 degrees
- moved R7 5.50 mm to (135.6, 74.8)
- moved C6 0.40 mm to (122.8, 78.5)
- moved R4 0.40 mm to (121.2, 78.5), turned to 90 degrees
Connections:
- C2 pad 2: /GNDIN -> GND
- DD1 pad 25: /T_SWDIO_IN -> /T_JTMS
- DD1 pad 38: (no net) -> /USB_RENUM
- R1 pad 1: /T_SWDIO_IN -> /USB_RENUM
- R1 pad 2: /T_JTMS -> +3v3
- R2 pad 1: /5VIN -> +5v
- R4 pad 1: +3v3 -> /USB_D+
- R4 pad 2: /USB_D+ -> Net-(Q1-Pad2)
- XL1 pad 1: /5VIN -> +5v
- XL1 pad 4: /GNDIN -> GND
- XL1 pad 5: /GNDIN -> GND
Routing:
- net GND: track 252.6 -> 146.0 mm, vias 52 -> 78
- net /5VIN: track 11.6 -> 0.00 mm, vias 2 -> 0
- net /GNDIN: track 10.5 -> 0.00 mm
- net +5v: track 8.39 -> 15.0 mm
- net Net-(Q1-Pad2): track 0.00 -> 6.18 mm
- net /USB_RENUM: track 0.00 -> 5.26 mm
- net /RXD: track 30.7 -> 26.6 mm, vias 4 -> 3
- net +3v3: track 78.6 -> 74.7 mm, vias 5 -> 4
- net /STM_JTCK: track 6.37 -> 8.80 mm
- net /T_SWDIO_IN: track 2.19 -> 0.00 mm
- net /AIN1: track 18.5 -> 17.6 mm
- net /STM_JTMS: track 11.9 -> 12.8 mm
- net /TXD: track 17.0 -> 16.2 mm
- net Net-(C11-Pad1): track 11.7 -> 11.0 mm
- net /T_JTCK: track 22.7 -> 22.1 mm
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Other:
- net class Default: via_dia 0.7 -> 0.6
- net class Wide: clearance 0.2 -> 0.15; via_dia 0.7 -> 0.6
- rule via_min_size: 0.4 -> 0.3
- board text added: "+3v3"
- board text added: "Ext Pwr On/Off"
- board text added: "GND"
- board text added: "Ostranna Teco v4"
- board text added: "RX"
- board text added: "SWCLK"
- board text added: "SWDIO"
- board text added: "TX"
- board text removed: "+ SWCLK GND SWDIO RX TX"
- board text removed: "Btn: Ext Pwr On/Off"
- board text removed: "Ostranna Teco v3"

Commit message: switch to KiCAD 7
Other:
- net class Default removed
- net class Wide removed

Commit message: USB-C connector installed, ESD USB protection added, new BOM created
Parts:
- removed XL1: USB_MICRO_2H, Connectors:USBmicro_MOLEX_1050170001
- added R8: 5.1k, Resistors:RES0603, F.Cu at (116.8, 84.5)
- added R9: 5.1k, Resistors:RES0603, F.Cu at (116.8, 81.4)
- added VD1: CM1213A−02SR, SOT,_TO:SOT143, F.Cu at (121.2, 83.0)
- added XS1: USBC 16PF-015, Connectors:USB-C_16pin_16PF-015, B.Cu at (118.6, 83.0)
- moved L1 2.07 mm to (122.5, 81.1), turned to 0 degrees
Connections:
- DD1 pad 11: (no net) -> unconnected-(DD1-ADC1-1/T2C2/PA1-Pad11)
- DD1 pad 14: (no net) -> unconnected-(DD1-ADC1-4/DAC1/CK2/PA4-Pad14)
- DD1 pad 16: (no net) -> unconnected-(DD1-ADC1-6/T3C1/MISO1/PA6-Pad16)
- DD1 pad 17: (no net) -> unconnected-(DD1-ADC1-7/T3C2/MOSI1/PA7-Pad17)
- DD1 pad 19: (no net) -> unconnected-(DD1-PB1/T3C4/ADC1-9-Pad19)
- DD1 pad 2: (no net) -> unconnected-(DD1-TAMPER-RTC/PC13-Pad2)
- DD1 pad 21: (no net) -> unconnected-(DD1-PB10/SCL2/TX3-Pad21)
- DD1 pad 22: (no net) -> unconnected-(DD1-PB11/SDA2/RX3-Pad22)
- DD1 pad 28: (no net) -> unconnected-(DD1-PB15/MOSI2/T1C3N/(T15C2)-Pad28)
- DD1 pad 29: (no net) -> unconnected-(DD1-T1C1/CK1/PA8-Pad29)
- DD1 pad 3: (no net) -> unconnected-(DD1-OC32IN/PC14-Pad3)
- DD1 pad 39: (no net) -> unconnected-(DD1-PB3/JTDO/(T2C2)-Pad39)
- DD1 pad 4: (no net) -> unconnected-(DD1-OC32OUT/PC15-Pad4)
- DD1 pad 40: (no net) -> unconnected-(DD1-PB4/JTRST/(T3C1)-Pad40)
- DD1 pad 41: (no net) -> unconnected-(DD1-PB5/(T3C2)-Pad41)
- DD1 pad 42: (no net) -> unconnected-(DD1-PB6/SCL1/T4C1/T16C1N-Pad42)
- DD1 pad 43: (no net) -> unconnected-(DD1-PB7/SDA1/T4C2/T17C1N-Pad43)
- DD1 pad 45: (no net) -> unconnected-(DD1-PB8/T4C3/T16C1-Pad45)
- DD1 pad 46: (no net) -> unconnected-(DD1-PB9/T4C4/T17C1-Pad46)
- DD1 pad 7: (no net) -> unconnected-(DD1-NRST-Pad7)
Routing:
- net GND: track 146.0 -> 132.4 mm, vias 78 -> 72
- net /USB_D+: track 6.16 -> 0.00 mm
- net +5v: track 15.0 -> 8.94 mm, vias 0 -> 1
- net /USB_D-: track 3.64 -> 0.00 mm
- net /USB_DIN-: track 3.40 -> 0.00 mm
- net Net-(XL1-PadH1): track 3.16 -> 0.00 mm
- net /USB_DIN+: track 3.12 -> 0.00 mm
- net +3v3: track 74.7 -> 74.1 mm

Commit message: upgrade complete
Parts:
- D1, D2: value LED -> LED G
- D3: value LED -> LED B
- DA1: value LD1117 -> LD1117S33
- moved R9 0.76 mm to (116.0, 81.5)
- moved R8 0.75 mm to (116.0, 84.5)
Routing:
- net GND: track 132.4 -> 150.2 mm, vias 72 -> 84
- net unconnected-(XS1-PadSHLD): track 0.00 -> 17.2 mm
- net +5v: track 8.94 -> 22.2 mm, vias 1 -> 2
- net /USB_DIN+: track 0.00 -> 7.31 mm, vias 0 -> 1
- net /USB_DIN-: track 0.00 -> 7.07 mm, vias 0 -> 1
- net /USB_D+: track 0.00 -> 4.26 mm
- net +3v3: track 74.1 -> 77.3 mm
- net /USB_CC2: track 0.00 -> 2.60 mm, vias 0 -> 1
- net /USB_CC1: track 0.00 -> 2.55 mm, vias 0 -> 1
- net /USB_D-: track 0.00 -> 1.58 mm
Other:
- rule pad_to_mask_clearance: 0.06 -> 0
- board text added: "Ostranna Teco v4.1"
- board text removed: "B"
- board text removed: "G"
- board text removed: "Ostranna Teco v4"
